File: Newer hotness/NH_PCB_V3/NH_PCB.kicad_pcb (KiCad board)
At the start: 2 copper layers, 96.5 x 63.5 mm, 16 parts, among them J1 CONN_02X03, J2 CONN_2_gnd, J3 POW_BYP, J4 BARREL_JACK, J5 SPI_debug, J6 I2C_Debug, U1 Teensy3.5, U2 ACCL_BOB_A1413, U3 10DOF_A1604

Commit message: updated v4 pcb
Parts:
- added G***: LOGO, logos:aiaa_logo_35in_fSS, F.Cu at (116.0, 124.2)
- added G***: LOGO, logos:aiaa_logo_inverse_2in_bSS, F.Cu at (129.9, 108.3)
- J4: footprint Connectors:BARREL_JACK -> custom_master:BARREL_JACK_W_Header_Holes
- renumbered REF** to ?
Routing:
- net /TX_STRAT: track 100.5 -> 110.7 mm, vias 2 -> 1
- net /5V: track 193.5 -> 200.4 mm
Other:
- board text added: "A1604"
- board text added: "Accel - A1430 +- 200g"
- board text added: "JARVIS V 1.1"
- board text added: "Teensy 3.5"
- board text removed: "3.5"
