File: Newer hotness/NH_PCB_V3/NH_PCB.sch (KiCad schematic (older format))
At the start: 10 parts, among them J1 CONN_02X03, J2 CONN_02X05, J3 POW_BYP, J4 BARREL_JACK, J5 CONN_01X02, J6 CONN_01X02, U1 Teensy3.5, U2 ACCL_BOB_A1413

Commit message: added final newer hotness boards
Parts:
- removed CO1: CONN_JST_2Pin, Connectors_JST:JST_PH_S2B-PH-SM4-TB_02x2.00mm_Angled, symbol CONN_JST_2Pin
- removed J2: CONN_02X05, Connectors:IDC_Header_Straight_10pins, symbol CONN_02X05
- added J2: CONN_2_gnd, Connectors_JST:JST_PH_S2B-PH-SM4-TB_02x2.00mm_Angled, symbol CONN_2_gnd
- added TC1, TC2: TCA-ADA-269, adafruit_BOBs:TCA_BOB_ADA269, symbol TCA-ADA-269
- added U3: 10DOF_A1604, adafruit_BOBs:10DOF_BOB_ADA16014, symbol 10DOF_A1604
- J5: value CONN_01X02 -> SPI_debug
- J6: value CONN_01X02 -> I2C_Debug
Connections:
- net TX_GPS is gone; now on net TX-GPS: J1.1 (P1)
- net 5V: now also TC1.1 (Vin), TC2.1 (Vin), U3.1 (Vin)
- net CLK: now also TC1.6 (CLK), TC2.6 (CLK)
- net CS-TC1: now also TC1.5 (CS)
- net CS_TS2: now also TC2.5 (CS)
- net DIN: now also U1.14 (12_MISO0), TC1.4 (DO), TC2.4 (DO); no longer U1.13 (11_MOSI0)
- net DOUT: now also U1.13 (11_MOSI0); no longer U1.14 (12_MISO0)
- net SCL: now also U3.4 (SCL_5V)
- net SDA: now also U3.5 (SDA_5V)
- net TX_STRAT: now also J2.1 (P1)
- net at U1.33 (36_A17_PWM): now also U3.9 (LSM_INT2)
- net at U1.34 (37_A18_PWM_SCL1): now also U3.10 (LSM_DRDY)
- net GIN: no longer names the net of U1.30 (33_A14_CAN1TX_scl0)
- net GIN: now also U3.6 (GYR_INT)
- net GIND: no longer names the net of U1.31 (34_A15_CAN1TX_sda0)
- net GIND: now also U3.7 (GRY_RDY)
- net GND_ renamed GND
- net GND: now also J2.2 (P2), TC1.3 (GND), TC2.3 (GND), U3.3 (GN)
- net XTRA: no longer names the net of U1.32 (35_A16_PWM)
- net XTRA: now also U3.8 (LSM_INT1)
- no-connect marks 1 -> 69
Other:
- note removed: "From 10DOF\nD-SUB-9"
- moved on the sheet: J1, J3

Commit message: updated v4 pcb
Parts:
- J4: footprint Connectors:BARREL_JACK -> custom_master:BARREL_JACK_W_Header_Holes
Changed lines of the file:
@@
 F 0 "J4" H 6450 1845 50  0000 C CNN
 F 1 "BARREL_JACK" H 6450 1495 50  0000 C CNN
-F 2 "Connectors:BARREL_JACK" H 6450 1650 50  0001 C CNN
+F 2 "custom_master:BARREL_JACK_W_Header_Holes" H 6450 1650 50  0001 C CNN
 F 3 "" H 6450 1650 50  0001 C CNN
 	1    6450 1650
