File: Newer hotness/NH_PCB_V4/NH_PCB.sch (KiCad schematic (older format))
At the start: 24 parts, among them J1 Xbee-Conn, J2 STRAT_CONN, J3 Pow_byp, J4 BARREL_JACK, J5 SPI_debug, J6 I2C_Debug, U1 Teensy3.6, U2 ACCL_BOB_A1413, U3 10DOF_A1604

Commit message: telemetry PCB updates
Connections:
- net CLK: now also J1.8 (P8)
- net Xbee_SS: now reaches U1.42 (15_A1_CS0_Touch)
- net Xbee_SS: now also J1.9 (P9)
- net Xbee_1 renamed GPS-FIX
- net Xbee_2 renamed Xbee_ATTN
- net Xbee_ATTN: now also J1.10 (P10); no longer J1.8 (P8)
- net Xbee_3: no longer names the net of U1.18 (26_tx1)
- net Xbee_3: no longer J1.9 (P9)
- net Xbee_4: no longer names the net of U1.19 (27_rx1)
- net Xbee_4: no longer J1.10 (P10)
- no-connect marks 64 -> 65
Other:
- moved on the sheet: TC1
Changed lines of the file:
@@
 L TCA-ADA-269 TC1
 U 1 1 596244C7
-P 4600 3600
-F 0 "TC1" H 4550 3450 60  0000 C CNN
-F 1 "TCA-ADA-269" H 4600 4350 60  0000 C CNN
-F 2 "adafruit_BOBs:TCA_BOB_ADA269" H 4600 3600 60  0001 C CNN
-F 3 "" H 4600 3600 60  0001 C CNN
-	1    4600 3600
+P 4600 3700
+F 0 "TC1" H 4550 3550 60  0000 C CNN
+F 1 "TCA-ADA-269" H 4600 4450 60  0000 C CNN
+F 2 "adafruit_BOBs:TCA_BOB_ADA269" H 4600 3700 60  0001 C CNN
+F 3 "" H 4600 3700 60  0001 C CNN
+	1    4600 3700
 	0    -1   1    0
 $EndComp
@@
 NoConn ~ 8600 3450
 NoConn ~ 8600 3550
-NoConn ~ 6600 5550
+NoConn ~ 6600 3150
 NoConn ~ 6600 5250
 NoConn ~ 6600 5050
@@
 	1    0    0    -1
 $EndComp
-Text Label 5350 3000 0    60   ~ 0
+Text Label 5350 3100 0    60   ~ 0
 3.3V
 NoConn ~ 4000 2150
-NoConn ~ 4000 3200
+NoConn ~ 4000 3300
 Text Label 8850 4550 0    60   ~ 0
 3.3V
@@
 	8950 5650 8600 5650
 Wire Wire Line
-	4200 2150 4200 3200
-Wire Wire Line
-	4300 2150 4300 3200
-Wire Wire Line
-	4500 2150 4500 3200
+	4200 2150 4200 3300
+Wire Wire Line
+	4300 2150 4300 3300
+Wire Wire Line
+	4500 2150 4500 3300
 Connection ~ 4200 2400
 Wire Wire Line
@@
 	4400 2350 4400 2150
 Wire Wire Line
-	4400 2500 4400 3200
+	4400 2500 4400 3300
 Wire Wire Line
 	6150 4450 6600 4450
@@
 	1800 2400 4200 2400
 Wire Wire Line
-	4100 2150 4100 3200
+	4100 2150 4100 3300
 Wire Wire Line
 	6250 3950 6150 3950
 Wire Wire Line
-	3550 3000 6250 3000
+	3550 3100 6250 3100
 Wire Wire Line
 	9150 4550 8600 4550
@@
 $EndComp
 Wire Wire Line
-	6250 3000 6250 3950
+	6250 3100 6250 3950
 $Comp
 L CONN_01X03 J3
@@
 3.3V
 Wire Wire Line
-	3550 3000 3550 2500
+	3550 3100 3550 2500
 Connection ~ 3550 2500
 $Comp
@@
 L PWR_FLAG #FLG05
 U 1 1 596CF3AC
-P 3800 3000
-F 0 "#FLG05" H 3800 3075 50  0001 C CNN
-F 1 "PWR_FLAG" H 3800 3150 50  0000 C CNN
-F 2 "" H 3800 3000 50  0001 C CNN
-F 3 "" H 3800 3000 50  0001 C CNN
-	1    3800 3000
-	1    0    0    -1
-$EndComp
-Connection ~ 3800 3000
+P 3800 3100
+F 0 "#FLG05" H 3800 3175 50  0001 C CNN
+F 1 "PWR_FLAG" H 3800 3250 50  0000 C CNN
+F 2 "" H 3800 3100 50  0001 C CNN
+F 3 "" H 3800 3100 50  0001 C CNN
+	1    3800 3100
+	1    0    0    -1
+$EndComp
+Connection ~ 3800 3100
 $Comp
 L PWR_FLAG #FLG06
@@
 Connection ~ 4100 4950
 Text Label 4250 6600 2    60   ~ 0
-Xbee_1
+GPS-FIX
 Text Label 4750 6600 0    60   ~ 0
-Xbee_2
+CLK
 Text Label 4250 6700 2    60   ~ 0
-Xbee_3
+Xbee_SS
 Text Label 4750 6700 0    60   ~ 0
-Xbee_4
+Xbee_ATTN
 Text Label 6600 2950 2    60   ~ 0
-Xbee_1
+GPS-FIX
 Text Label 6600 3050 2    60   ~ 0
-Xbee_2
-Text Label 6600 3150 2    60   ~ 0
-Xbee_3
-Text Label 6600 3250 2    60   ~ 0
-Xbee_4
+Xbee_ATTN
+Text Label 6600 5550 2    60   ~ 0
+Xbee_SS
 $Comp
 L L7805AC REG1
@@
 Wire Wire Line
 	6450 3850 6600 3850
+NoConn ~ 6600 3250
+$Comp
+L PWR_FLAG #FLG09
+U 1 1 59767C02
+P 6250 5150
+F 0 "#FLG09" H 6250 5225 50  0001 C CNN
+F 1 "PWR_FLAG" H 6250 5300 50  0000 C CNN
+F 2 "" H 6250 5150 50  0001 C CNN
+F 3 "" H 6250 5150 50  0001 C CNN
+	1    6250 5150
+	1    0    0    -1
+$EndComp
+Connection ~ 6250 5150
 $EndSCHEMATC

Commit message: updated PCB files
Parts:
- added BZ1: Buzzer, adafruit_BOBs:Buzzer_A1536, symbol Buzzer
Connections:
- net GND: now also BZ1.2 (+)
- net at U1.47 (20_A6_PWM_CS0_sck1): now also BZ1.1 (-)
- no-connect marks 65 -> 64
Changed lines of the file:
@@
 NoConn ~ 8600 4450
 NoConn ~ 8600 5050
-NoConn ~ 8600 5350
 NoConn ~ 8600 4950
 NoConn ~ 9300 4750
@@
 $EndComp
 Connection ~ 6250 5150
+$Comp
+L Buzzer BZ1
+U 1 1 597B84D0
+P 9200 5900
+F 0 "BZ1" H 9350 5950 50  0000 L CNN
+F 1 "Buzzer" H 9350 5850 50  0000 L CNN
+F 2 "adafruit_BOBs:Buzzer_A1536" V 9175 6000 50  0001 C CNN
+F 3 "" V 9175 6000 50  0001 C CNN
+	1    9200 5900
+	1    0    0    -1
+$EndComp
+$Comp
+L GND #PWR010
+U 1 1 597B894B
+P 8850 6200
+F 0 "#PWR010" H 8850 5950 50  0001 C CNN
+F 1 "GND" H 8850 6050 50  0000 C CNN
+F 2 "" H 8850 6200 50  0001 C CNN
+F 3 "" H 8850 6200 50  0001 C CNN
+	1    8850 6200
+	1    0    0    -1
+$EndComp
+Wire Wire Line
+	8600 5350 8850 5350
+Wire Wire Line
+	8850 5350 8850 5800
+Wire Wire Line
+	8850 5800 9100 5800
+Wire Wire Line
+	9100 6000 8850 6000
+Wire Wire Line
+	8850 6000 8850 6200
 $EndSCHEMATC

Commit message: Finalized NH PCBs
Parts:
- added J7: Pow_in, Pin_Headers:Pin_Header_Straight_1x02, symbol CONN_01X02
Connections:
- net GND: now also J7.2 (P2)
- net at C3.1, J4.1, REG1.1 (Vin): now also J7.1 (P1)
Other:
- note removed: "4"
- note removed: "Adam Poirier"
- note removed: "Northeastern AIAA\nProject Karman telemetry system\nVersion 2, Rev 4"
Changed lines of the file:
@@
 encoding utf-8
 Sheet 1 1
-Title ""
-Date ""
-Rev ""
-Comp ""
+Title "JARVIS 2.0 - MCU"
+Date "2017-07-31"
+Rev "5"
+Comp "AIAA Northeastern - Project Karman"
 Comment1 ""
-Comment2 ""
-Comment3 ""
-Comment4 ""
+Comment2 "Adam Poirier"
+Comment3 "Primary board - MCU module (board 1 / 2)"
+Comment4 "Project Karman Telemetry System "
 $EndDescr
 $Comp
@@
 L PWR_FLAG #FLG01
 U 1 1 5964E87C
-P 4100 4650
-F 0 "#FLG01" H 4100 4725 50  0001 C CNN
-F 1 "PWR_FLAG" H 4100 4800 50  0000 C CNN
-F 2 "" H 4100 4650 50  0001 C CNN
-F 3 "" H 4100 4650 50  0001 C CNN
-	1    4100 4650
+P 4100 4200
+F 0 "#FLG01" H 4100 4275 50  0001 C CNN
+F 1 "PWR_FLAG" H 4100 4350 50  0000 C CNN
+F 2 "" H 4100 4200 50  0001 C CNN
+F 3 "" H 4100 4200 50  0001 C CNN
+	1    4100 4200
 	1    0    0    -1
 $EndComp
@@
 Wire Wire Line
 	2100 3150 2100 4650
-Text Notes 10400 7050 0    60   ~ 0
-Adam Poirier
-Text Notes 7000 6900 0    60   ~ 0
-Northeastern AIAA\nProject Karman telemetry system\nVersion 2, Rev 4
-Text Notes 10600 7650 0    60   ~ 0
-4
 Connection ~ 1800 5050
 Wire Wire Line
@@
 	3700 4650 4500 4650
 Wire Wire Line
-	2800 4950 4400 4950
-Wire Wire Line
-	4400 4950 4400 4850
+	4400 4950 2800 4950
+Wire Wire Line
+	4400 4300 4400 4950
 Wire Wire Line
 	4400 4850 4500 4850
 Connection ~ 3600 4950
 Wire Wire Line
-	2800 5050 2800 4950
+	2800 4950 2800 5050
 $Comp
 L C C3
@@
 Wire Wire Line
 	8850 6000 8850 6200
+$Comp
+L CONN_01X02 J7
+U 1 1 5983B429
+P 4800 4250
+F 0 "J7" H 4800 4400 50  0000 C CNN
+F 1 "Pow_in" V 4900 4250 50  0000 C CNN
+F 2 "Pin_Headers:Pin_Header_Straight_1x02" H 4800 4250 50  0001 C CNN
+F 3 "" H 4800 4250 50  0001 C CNN
+	1    4800 4250
+	1    0    0    -1
+$EndComp
+Wire Wire Line
+	4600 4200 4100 4200
+Wire Wire Line
+	4100 4200 4100 4650
+Connection ~ 4100 4200
+Wire Wire Line
+	4600 4300 4400 4300
+Connection ~ 4400 4850
 $EndSCHEMATC
