File: Newer hotness/Xbee_GPS/Xbee_GPS.kicad_pcb (KiCad board)
At the start: 2 copper layers, 50.8 x 76.2 mm, 22 parts, among them J1 BARREL_JACK, J2 CONN_02X05, J3 GS3, J4 FTDI_Header, J5 GS3

Commit message: updated PCB files
Parts:
- added G***: LOGO, logos:aiaa_logo_inverse_2in_bSS, F.Cu at (125.5, 75.3)
- 3.3V Regulator: renamed from regul1
- FTDI Header: renamed from J4
- moved C3 5.33 mm to (106.9, 38.1)
- moved C1 5.03 mm to (107.0, 43.1)
Routing:
- net GND: track 131.2 -> 110.4 mm
- net /TX-XB: track 61.9 -> 63.1 mm
Other:
- net class Default: via_dia 0.6 -> 0.762
- rule pad_to_mask_clearance: 0.2 -> 0.2032
- rule via_min_size: 0.4 -> 0.635
- board text added: "10µF"
- board text added: "47pF"
- board text added: "5 - 15 Vin"
- board text added: "FTDI POW"
- board text added: "GND"
- board text added: "GREEN"
- board text added: "MOSI"
- board text added: "MSIO"
- board text added: "NU AIAA Project Karman Adam Poirier"
- board text added: "NU AIAA Project Karman Adam Poirier Telemetry Transmitter Module JARVIS V2.0"
- board text added: "Serial - Top pads SPI - Bottom pads"
- board text added: "X-RX"
- board text added: "X-TX"

Commit message: Finalized NH PCBs
Parts:
- added J6: Pow_conn, Pin_Headers:Pin_Header_Straight_1x02, F.Cu at (136.6, 106.0)
- J4: renamed from FTDI Header
- regul1: renamed from 3.3V Regulator
- moved G*** 28.6 mm to (109.0, 106.4)
Routing:
- net /PWR: track 21.3 -> 25.5 mm
Other:
- board text added: "+ -"
- board text added: "Power"
Changed lines of the file:
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@@
 (kicad_pcb (version 4) (host pcbnew 4.0.6)
   (general
-    (links 41)
+    (links 43)
     (no_connects 0)
     (area 96.8502 17.758999 150.241001 111.633001)
     (thickness 1.6)
-    (drawings 20)
-    (tracks 217)
+    (drawings 22)
+    (tracks 219)
     (zones 0)
-    (modules 23)
+    (modules 24)
     (nets 34)
   )
@@
   )
   (setup
-    (last_trace_width 0.25)
+    (last_trace_width 0.762)
     (user_trace_width 0.762)
     (trace_clearance 0.2)
@@
     (descr "Through hole straight pin header, 1x06, 2.54mm pitch, single row")
     (tags "Through hole pin header THT 1x06 2.54mm single row")
-    (fp_text reference "FTDI Header" (at -2.5654 5.0038 450) (layer F.SilkS)
+    (fp_text reference J4 (at -2.5654 5.0038 450) (layer F.SilkS)
       (effects (font (size 1 1) (thickness 0.15)))
     )
@@
     (descr "TO-220, Neutral, Vertical,")
     (tags "TO-220, Neutral, Vertical,")
-    (fp_text reference "3.3V Regulator" (at 0 -4.572 90) (layer F.SilkS)
+    (fp_text reference regul1 (at 0 -4.572 90) (layer F.SilkS)
       (effects (font (size 1 1) (thickness 0.15)))
     )
@@
   )
   (module logos:aiaa_logo_35in_fSS (layer F.Cu)
-    (at 137.668 106.426)
+    (at 109.0422 106.3752)
     (fp_text reference G*** (at 0 0) (layer F.SilkS) hide
       (effects (font (thickness 0.3)))
@@
       (xy -8.720667 -18.647833)) (layer B.SilkS) (width 0.01))
   )
+  (module Pin_Headers:Pin_Header_Straight_1x02 (layer F.Cu)
+    (at 136.5504 106.0196 90)
+    (descr "Through hole pin header")
+    (tags "pin header")
+    (fp_text reference J6 (at 0.0508 4.6736 180) (layer F.SilkS)
+      (effects (font (size 1 1) (thickness 0.15)))
+    )
+    (fp_text value Pow_conn (at 0 -3.1 90) (layer F.Fab)
+      (effects (font (size 1 1) (thickness 0.15)))
+    )
+    (fp_line (start 1.27 1.27) (end 1.27 3.81) (layer F.SilkS) (width 0.15))
+    (fp_line (start 1.55 -1.55) (end 1.55 0) (layer F.SilkS) (width 0.15))
+    (fp_line (start -1.75 -1.75) (end -1.75 4.3) (layer F.CrtYd) (width 0.05))
+    (fp_line (start 1.75 -1.75) (end 1.75 4.3) (layer F.CrtYd) (width 0.05))
+    (fp_line (start -1.75 -1.75) (end 1.75 -1.75) (layer F.CrtYd) (width 0.05))
+    (fp_line (start -1.75 4.3) (end 1.75 4.3) (layer F.CrtYd) (width 0.05))
+    (fp_line (start 1.27 1.27) (end -1.27 1.27) (layer F.SilkS) (width 0.15))
+    (fp_line (start -1.55 0) (end -1.55 -1.55) (layer F.SilkS) (width 0.15))
+    (fp_line (start -1.55 -1.55) (end 1.55 -1.55) (layer F.SilkS) (width 0.15))
+    (fp_line (start -1.27 1.27) (end -1.27 3.81) (layer F.SilkS) (width 0.15))
+    (fp_line (start -1.27 3.81) (end 1.27 3.81) (layer F.SilkS) (width 0.15))
+    (pad 1 thru_hole rect (at 0 0 90) (size 2.032 2.032) (drill 1.016) (layers *.Cu *.Mask)
+      (net 33 /PWR))
+    (pad 2 thru_hole oval (at 0 2.54 90) (size 2.032 2.032) (drill 1.016) (layers *.Cu *.Mask)
+      (net 3 GND))
+    (model Pin_Headers.3dshapes/Pin_Header_Straight_1x02.wrl
+      (at (xyz 0 -0.05 0))
+      (scale (xyz 1 1 1))
+      (rotate (xyz 0 0 90))
+    )
+  )
+  (gr_text Power (at 137.7696 103.6066) (layer F.SilkS)
+    (effects (font (size 0.992 0.992) (thickness 0.15)))
+  )
+  (gr_text "+   -" (at 137.8712 108.3818) (layer F.SilkS)
+    (effects (font (size 0.992 0.992) (thickness 0.15)))
+  )
   (gr_text "FTDI POW" (at 130.4798 95.4786) (layer F.SilkS)
     (effects (font (size 0.508 0.508) (thickness 0.127)))
@@
   (segment (start 114.533842 45.212) (end 119.257 45.212) (width 0.25) (layer F.Cu) (net 32))
   (segment (start 119.257 45.212) (end 120.142 45.212) (width 0.25) (layer F.Cu) (net 32))
+  (segment (start 132.3848 106.0958) (end 136.4742 106.0958) (width 0.762) (layer F.Cu) (net 33) (status C00000))
+  (segment (start 136.4742 106.0958) (end 136.5504 106.0196) (width 0.762) (layer F.Cu) (net 33) (status C00000))
   (segment (start 122.7836 103.8606) (end 122.7836 99.81946) (width 0.762) (layer F.Cu) (net 33))
   (segment (start 122.7836 99.81946) (end 120.396 97.43186) (width 0.762) (layer F.Cu) (net 33))

Commit message: making sure up to date
Parts:
- added D3: LED, LEDs:LED-3MM, F.Cu at (124.9, 92.6)
- added R1: 100, Resistors_THT:R_Axial_DIN0207_L6.3mm_D2.5mm_P7.62mm_Horizontal, F.Cu at (127.4, 91.8)
- moved JP1 2.21 mm to (127.9, 95.1)
Routing:
- net +3V3: track 107.0 -> 72.8 mm, vias 1 -> 0
- net GND: track 110.4 -> 123.6 mm, vias 2 -> 1
- net /Vbat: track 35.4 -> 46.0 mm, vias 1 -> 0
- net /RX-GPS: track 53.6 -> 45.3 mm, vias 0 -> 1
- net /TX_GPS: track 58.1 -> 52.1 mm
- net Net-(D3-Pad1): track 0.00 -> 2.85 mm
- net /GPS-FIX: track 48.0 -> 46.4 mm
- net Net-(D2-Pad2): track 14.0 -> 12.4 mm
- net Net-(J4-Pad3): track 45.3 -> 45.9 mm
