File: Newer hotness/Xbee_GPS/Xbee_GPS.sch (KiCad schematic (older format))
At the start: 15 parts, among them J1 BARREL_JACK, J2 CONN_02X05, J3 GS3, J4 FTDI_Header, J5 GS3

Commit message: updated PCB files
Changed lines of the file:
@@
 EESchema Schematic File Version 2
+LIBS:NH_PCB-rescue
 LIBS:power
 LIBS:device
@@
 LIBS:contrib
 LIBS:valves
+LIBS:teensy
+LIBS:adafruit_BOBs
 LIBS:master_custom
-LIBS:adafruit_BOBs
-LIBS:Xbee_GPS-cache
+LIBS:NH_PCB-cache
 EELAYER 25 0
 EELAYER END
@@
 	1    0    0    -1
 $EndComp
-Wire Wire Line
-	3350 3250 2600 3250
-Wire Wire Line
-	3350 2600 3350 4550
-Wire Wire Line
-	3350 4000 5600 4000
-Wire Wire Line
-	3700 3350 2600 3350
-Wire Wire Line
-	1650 3350 2100 3350
 Text Label 7500 3900 0    60   ~ 0
 CTS-XB
@@
 	1    0    0    -1
 $EndComp
-Wire Wire Line
-	3250 3100 5600 3100
-Connection ~ 5150 3100
-Connection ~ 4850 3100
-Connection ~ 5150 2800
 $Comp
 L LD1117V33 regul1
@@
 	0    -1   1    0
 $EndComp
-Connection ~ 4850 2800
 $Comp
 L BARREL_JACK J1
@@
 	1    0    0    -1
 $EndComp
-Connection ~ 3350 3250
-Connection ~ 3350 2800
 $Comp
 L GPS_BOB_ADA-746 BOB1
@@
 	1    0    0    -1
 $EndComp
-Wire Wire Line
-	2900 4450 3000 4450
-Wire Wire Line
-	3000 4450 3000 4150
-Wire Wire Line
-	3000 4150 1700 4150
-Wire Wire Line
-	1700 4150 1700 3450
-Wire Wire Line
-	1700 3450 2100 3450
-Wire Wire Line
-	2100 3250 1500 3250
-Wire Wire Line
-	1500 3250 1500 4850
-Wire Wire Line
-	1500 4850 2000 4850
-Wire Wire Line
-	2000 4750 1600 4750
-Wire Wire Line
-	1600 4750 1600 3550
-Wire Wire Line
-	1600 3550 2100 3550
 $Comp
 L Battery_Cell BT1
@@
 Text Label 7700 1350 0    60   ~ 0
 Vbat
-Wire Wire Line
-	7500 1500 7500 1350
-Wire Wire Line
-	7500 1350 7700 1350
 $Comp
 L GND #PWR01
@@
 	1    0    0    -1
 $EndComp
-Connection ~ 2450 2800
-Wire Wire Line
-	3350 4550 2900 4550
-Connection ~ 3350 4000
-Wire Wire Line
-	7500 1800 7500 2000
 $Comp
 L +3.3V #PWR03
@@
 	1    0    0    -1
 $EndComp
-Wire Wire Line
-	2000 4450 1900 4450
-Wire Wire Line
-	1900 4450 1900 4050
-Wire Wire Line
-	1900 4050 3250 4050
-Connection ~ 2850 4050
 $Comp
 L PWR_FLAG #FLG04
@@
 	1    0    0    -1
 $EndComp
-Connection ~ 2450 2600
 Text Label 2000 4650 2    60   ~ 0
 Vbat
@@
 	-1   0    0    1
 $EndComp
-Wire Wire Line
-	3700 3350 3700 3750
-Wire Wire Line
-	3700 3750 4500 3750
-Wire Wire Line
-	4800 3650 4900 3650
-Wire Wire Line
-	4900 3650 4900 3300
-Wire Wire Line
-	4450 3300 5600 3300
-Wire Wire Line
-	4200 3200 5600 3200
-Wire Wire Line
-	3800 3300 3900 3300
-Wire Wire Line
-	7200 4000 7200 4350
-Wire Wire Line
-	7200 4350 4450 4350
-Wire Wire Line
-	4450 4350 4450 3400
-Wire Wire Line
-	4450 3400 4200 3400
-Wire Wire Line
-	5000 3400 5600 3400
-Wire Wire Line
-	5000 3400 5000 3850
-Wire Wire Line
-	5000 3850 4800 3850
 Text Label 7200 3300 0    60   ~ 0
 Xbee_CLK
@@
 NoConn ~ 2900 4650
 NoConn ~ 1700 2700
-Wire Wire Line
-	7450 3700 7450 4050
 $Comp
 L GND #PWR05
@@
 	1    0    0    -1
 $EndComp
-Wire Wire Line
-	3250 4050 3250 2600
-Wire Wire Line
-	1650 3350 1650 3800
-Wire Wire Line
-	1650 3800 3800 3800
-Wire Wire Line
-	3800 3800 3800 3300
-Connection ~ 3250 3100
-Wire Wire Line
-	1700 2800 5450 2800
 $Comp
 L CONN_01X06 J4
@@
 Text Notes 3650 1200 0    60   ~ 0
 Black
-Wire Wire Line
-	4150 1350 4150 2800
-Connection ~ 4150 2800
-Wire Wire Line
-	4250 1350 4250 2500
-Wire Wire Line
-	4250 2500 7950 2500
-Wire Wire Line
-	7950 2500 7950 3900
-Wire Wire Line
-	4350 1350 4350 1700
-Wire Wire Line
-	2750 1700 2750 1900
 $Comp
 L D_Shockley D2
@@
 	-1   0    0    1
 $EndComp
-Wire Wire Line
-	2750 2600 2750 2200
-Connection ~ 2750 2600
-Wire Wire Line
-	1700 2600 1900 2600
-Wire Wire Line
-	2200 2600 3150 2600
 $Comp
 L Jumper JP1
@@
 	1    0    0    -1
 $EndComp
-Wire Wire Line
-	4350 1700 3750 1700
-Wire Wire Line
-	3150 1700 2750 1700
-Wire Wire Line
-	4450 1350 4450 3300
-Connection ~ 4900 3300
 Text Label 4900 3300 0    60   ~ 0
 TX_EX
 Text Label 5150 3200 0    60   ~ 0
 RX_EX
-Connection ~ 5450 3100
-Wire Wire Line
-	4550 1350 4550 3200
-Connection ~ 4550 3200
-Wire Wire Line
-	7200 3700 7450 3700
-Wire Wire Line
-	7950 3900 7200 3900
-Wire Wire Line
-	7200 3500 7850 3500
-Wire Wire Line
-	7850 3500 7850 2600
-Wire Wire Line
-	7850 2600 4650 2600
-Wire Wire Line
-	4650 2600 4650 1350
 Text Notes 4700 1900 0    60   ~ 0
 1 (Black) - pin 10 ground\n2 (Brown) - pin 12 cts\n3 (Red) - 5V - VCC (convert to 3.3)\n4 (Orange) - pin 3 tx to din\n5 (Yellow) - pin 2 rx to dout\n6 (Green) - pin 16 rts
@@
 Text Label 1750 2600 0    60   ~ 0
 PWR
+Wire Wire Line
+	3350 3250 2600 3250
+Wire Wire Line
+	3350 2600 3350 2800
+Wire Wire Line
+	3350 2800 3350 3250
+Wire Wire Line
+	3350 3250 3350 4000
+Wire Wire Line
+	3350 4000 3350 4550
+Wire Wire Line
+	3350 4000 5600 4000
+Wire Wire Line
+	3700 3350 2600 3350
+Wire Wire Line
+	1550 3350 2100 3350
+Wire Wire Line
+	3250 3100 4850 3100
+Wire Wire Line
+	4850 3100 5150 3100
+Wire Wire Line
+	5150 3100 5450 3100
+Wire Wire Line
+	5450 3100 5600 3100
+Connection ~ 5150 3100
+Connection ~ 4850 3100
+Connection ~ 5150 2800
+Connection ~ 4850 2800
+Connection ~ 3350 3250
+Connection ~ 3350 2800
+Wire Wire Line
+	2900 4450 3000 4450
+Wire Wire Line
+	3000 4450 3000 4150
+Wire Wire Line
+	3000 4150 1700 4150
+Wire Wire Line
+	1700 4150 1700 3450
+Wire Wire Line
+	1700 3450 2100 3450
+Wire Wire Line
+	2100 3250 1250 3250
+Wire Wire Line
+	1250 3250 1250 4850
+Wire Wire Line
+	1250 4850 2000 4850
+Wire Wire Line
+	2000 4750 1450 4750
+Wire Wire Line
+	1450 4750 1450 3550
+Wire Wire Line
+	1450 3550 2100 3550
+Wire Wire Line
+	7500 1500 7500 1350
+Wire Wire Line
+	7500 1350 7700 1350
+Connection ~ 2450 2800
+Wire Wire Line
+	3350 4550 2900 4550
+Connection ~ 3350 4000
+Wire Wire Line
+	7500 1800 7500 2000
+Wire Wire Line
+	2000 4450 1900 4450
+Wire Wire Line
+	1900 4450 1900 4050
+Wire Wire Line
+	1900 4050 2850 4050
+Wire Wire Line
+	2850 4050 3250 4050
+Connection ~ 2850 4050
+Connection ~ 2450 2600
+Wire Wire Line
+	3700 3350 3700 3750
+Wire Wire Line
+	3700 3750 4500 3750
+Wire Wire Line
+	4800 3650 4900 3650
+Wire Wire Line
+	4900 3650 4900 3300
+Wire Wire Line
+	4450 3300 4900 3300
+Wire Wire Line
+	4900 3300 5600 3300
+Wire Wire Line
+	4200 3200 4550 3200
+Wire Wire Line
+	4550 3200 5600 3200
+Wire Wire Line
+	3800 3300 3900 3300
+Wire Wire Line
+	7200 4000 7200 4350
+Wire Wire Line
+	7200 4350 4450 4350
+Wire Wire Line
+	4450 4350 4450 3400
+Wire Wire Line
+	4450 3400 4200 3400
+Wire Wire Line
+	5000 3400 5600 3400
+Wire Wire Line
+	5000 3400 5000 3850
+Wire Wire Line
+	5000 3850 4800 3850
+Wire Wire Line
+	7450 3700 7450 4050
+Wire Wire Line
+	3250 4050 3250 3100
+Wire Wire Line
+	3250 3100 3250 2600
+Wire Wire Line
+	1550 3350 1550 3800
+Wire Wire Line
+	1550 3800 3800 3800
+Wire Wire Line
+	3800 3800 3800 3300
+Connection ~ 3250 3100
+Wire Wire Line
+	1700 2800 2450 2800
+Wire Wire Line
+	2450 2800 3350 2800
+Wire Wire Line
+	3350 2800 4150 2800
+Wire Wire Line
+	4150 2800 4850 2800
+Wire Wire Line
+	4850 2800 5150 2800
+Wire Wire Line
+	5150 2800 5450 2800
+Wire Wire Line
+	4150 1350 4150 2800
+Connection ~ 4150 2800
+Wire Wire Line
+	4250 1350 4250 2500
+Wire Wire Line
+	4250 2500 7950 2500
+Wire Wire Line
+	7950 2500 7950 3900
+Wire Wire Line
+	4350 1350 4350 1700
+Wire Wire Line
+	2750 1700 2750 1900
+Wire Wire Line
+	2750 2600 2750 2200
+Connection ~ 2750 2600
+Wire Wire Line
+	1700 2600 1900 2600
+Wire Wire Line
+	2200 2600 2450 2600
+Wire Wire Line
+	2450 2600 2750 2600
+Wire Wire Line
+	2750 2600 3150 2600
+Wire Wire Line
+	4350 1700 3750 1700
+Wire Wire Line
+	3150 1700 2750 1700
+Wire Wire Line
+	4450 1350 4450 3300
+Connection ~ 4900 3300
+Connection ~ 5450 3100
+Wire Wire Line
+	4550 1350 4550 3200
+Connection ~ 4550 3200
+Wire Wire Line
+	7200 3700 7450 3700
+Wire Wire Line
+	7950 3900 7200 3900
+Wire Wire Line
+	7200 3500 7850 3500
+Wire Wire Line
+	7850 3500 7850 2600
+Wire Wire Line
+	7850 2600 4650 2600
+Wire Wire Line
+	4650 2600 4650 1350
 $EndSCHEMATC

Commit message: Finalized NH PCBs
Parts:
- added J6: Pow_conn, Pin_Headers:Pin_Header_Straight_1x02, symbol CONN_01X02
Connections:
- net GND: now also J6.2 (P2)
- net PWR: now also J6.1 (P1)
Other:
- moved on the sheet: BOB1, BT1, C1, C2, C3, D1, D2, J1, J2, J3, J4, J5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

Commit message: making sure up to date
Parts:
- added D3: LED, LEDs:LED-3MM, symbol LED
- added R1: 100, Resistors_THT:R_Axial_DIN0207_L6.3mm_D2.5mm_P7.62mm_Horizontal, symbol R
Connections:
- net GND: now also D3.2 (A), R1.2
- new net: D3.1 (K), R1.1
Changed lines of the file:
@@
 	3100 4100 3100 3800
 Connection ~ 3100 3800
+$Comp
+L LED D3
+U 1 1 59B311EE
+P 4550 5550
+F 0 "D3" H 4550 5650 50  0000 C CNN
+F 1 "LED" H 4550 5450 50  0000 C CNN
+F 2 "LEDs:LED-3MM" H 4550 5550 50  0001 C CNN
+F 3 "" H 4550 5550 50  0001 C CNN
+	1    4550 5550
+	-1   0    0    1
+$EndComp
+Connection ~ 4400 5550
+$Comp
+L GND #PWR06
+U 1 1 59B3129A
+P 4900 5850
+F 0 "#PWR06" H 4900 5600 50  0001 C CNN
+F 1 "GND" H 4900 5700 50  0000 C CNN
+F 2 "" H 4900 5850 50  0001 C CNN
+F 3 "" H 4900 5850 50  0001 C CNN
+	1    4900 5850
+	1    0    0    -1
+$EndComp
+Wire Wire Line
+	4900 5550 4700 5550
+$Comp
+L R R1
+U 1 1 59B3136C
+P 4900 5700
+F 0 "R1" V 4980 5700 50  0000 C CNN
+F 1 "100" V 4900 5700 50  0000 C CNN
+F 2 "Resistors_THT:R_Axial_DIN0207_L6.3mm_D2.5mm_P7.62mm_Horizontal" V 4830 5700 50  0001 C CNN
+F 3 "" H 4900 5700 50  0001 C CNN
+	1    4900 5700
+	1    0    0    -1
+$EndComp
 $EndSCHEMATC
